File: hardware/colorswitch/v0.4/colorswitch.kicad_pcb (KiCad board)
At the start: 2 copper layers, 96.7 x 44 mm, 49 parts, among them J1 Conn_02x05_Odd_Even, J2 Conn_01x06, J3 Conn_01x02_Pin, J4 DA15_Plug, J5 DA15_Plug, Q1 2N3904, Q2 2N3904, Q3 2N3904, Q4 2N3904, Q5 2N3904, Q6 2N3904, Q8 2N3906, U1 74LS241, U2 74LS08

Commit message: Add files via upload
Parts:
- moved R23 0.25 mm to (130.2, 105.7)
- moved R28 0.25 mm to (145.4, 105.7)
- moved R13 0.25 mm to (114.9, 105.8)
- moved R18 0.23 mm to (99.7, 105.7)
- moved R10 0.13 mm to (170.2, 110.5)
Routing:
- net CG: track 123.1 -> 124.3 mm
- net GND1: track 64.0 -> 62.8 mm
Other:
- board text added: "B"
- board text added: "G"
- board text added: "GND"
- board text added: "R"
- board text added: "SYN"
- board text added: "VCC"
